File: joint_pcb/joint_pcb.sch (KiCad schematic (older format))
At the start: 2 parts, among them J1 Conn_02x15_Odd_Even, J2 Conn_02x20_Odd_Even

Commit message: Replace to pin socket from pin header on join pcb
Parts:
- J1, J2: footprint Connector_PinHeader_2.54mm:PinHeader_2x20_P2.54mm_Vertical -> Connector_PinSocket_2.54mm:PinSocket_2x20_P2.54mm_Vertical
Changed lines of the file:
@@
 F 0 "J2" H 5600 3700 50  0000 C CNN
 F 1 "Conn_02x20_Odd_Even" H 5600 3600 50  0000 C CNN
-F 2 "Connector_PinHeader_2.54mm:PinHeader_2x20_P2.54mm_Vertical" H 5550 2600 50  0001 C CNN
+F 2 "Connector_PinSocket_2.54mm:PinSocket_2x20_P2.54mm_Vertical" H 5550 2600 50  0001 C CNN
 F 3 "~" H 5550 2600 50  0001 C CNN
 	1    5550 2600
@@
 F 0 "J1" H 5600 3700 50  0000 C CNN
 F 1 "Conn_02x15_Odd_Even" H 5600 3600 50  0000 C CNN
-F 2 "Connector_PinHeader_2.54mm:PinHeader_2x20_P2.54mm_Vertical" H 5550 2600 50  0001 C CNN
+F 2 "Connector_PinSocket_2.54mm:PinSocket_2x20_P2.54mm_Vertical" H 5550 2600 50  0001 C CNN
 F 3 "~" H 5550 2600 50  0001 C CNN
 	1    5550 2600
