File: main_pcb/main_pcb.sch (KiCad schematic (older format))
At the start: 7 parts, among them J1 Conn_01x17, J2 Conn_01x17, P1 Conn_02x20_Odd_Even

Commit message: Apply header footprints to main pcb
Parts:
- P1: footprint Connector_PinSocket_2.54mm:PinSocket_2x20_P2.54mm_Vertical -> Connector_PinHeader_2.54mm:PinHeader_2x20_P2.54mm_Vertical
Changed lines of the file:
@@
 F 0 "P1" H 7150 4767 50  0000 C CNN
 F 1 "Conn_02x20_Odd_Even" H 7150 4676 50  0000 C CNN
-F 2 "Connector_PinSocket_2.54mm:PinSocket_2x20_P2.54mm_Vertical" H 2250 2700 50  0001 C CNN
+F 2 "Connector_PinHeader_2.54mm:PinHeader_2x20_P2.54mm_Vertical" H 2250 2700 50  0001 C CNN
 F 3 "" H 2250 2700 50  0001 C CNN
 	1    7100 3650
